Commit message: Snapshot thesis research sources, paper materials and summaries
Include V2-V6 and PCT/TEB/DWA research materials, restoreable submodule patches, and the independent ASTRA source overlay. Keep raw experiment data, build outputs, runtime logs, and duplicate archives local.

File: src/simulation/m2_gazebo/urdf/m2_base.xacro (robot description, xacro)
@@ -25,5 +25,5 @@
         <material name="m2_tire"><color rgba="0.06 0.06 0.06 1"/></material>
       </visual>
-      <collision name="${prefix}chassis_collision">
+      <collision name="${prefix}${name}_wheel_collision">
         <origin rpy="${pi/2} 0 0"/>
         <geometry><cylinder radius="${wheel_radius}" length="${wheel_width}"/></geometry>
@@ -76,5 +76,5 @@
         <material name="m2_body"><color rgba="0.12 0.32 0.62 1"/></material>
       </visual>
-      <collision>
+      <collision name="${prefix}chassis_collision">
         <origin xyz="0 0 ${body_center_z}"/>
         <geometry><box size="${body_length} ${body_width} ${body_height}"/></geometry>
